File: Electronics/CanSat2023.kicad_pcb (KiCad board)
At the start: 2 copper layers, 42 parts, among them J1 Conn_01x02, J2 Conn_01x02, J3 Conn_01x06, J4 Conn_01x06, J5 Conn_01x06, J6 Conn_01x06, U1 NCP1117-3.3_SOT223, U2 W25Q128JVS, U3 RP2040, U4 A4950E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

Commit message: Correct files
Parts:
- removed J2: Conn_01x02, Connector_PinHeader_2.54mm:PinHeader_1x02_P2.54mm_Vertical
- added C3: 10u, Capacitor_SMD:C_0201_0603Metric, B.Cu at (41.1, 51.3)
- added C4: 10u, Capacitor_SMD:C_0201_0603Metric, B.Cu at (41.1, 56.4)
- added H1: MountingHole, MountingHole:MountingHole_4mm, F.Cu at (41.0, 15.2)
- added H2: MountingHole, MountingHole:MountingHole_4mm, F.Cu at (41.0, 67.0)
- added H3: MountingHole, MountingHole:MountingHole_4mm, F.Cu at (67.0, 41.0)
- added H4: MountingHole, MountingHole:MountingHole_4mm, F.Cu at (15.2, 41.0)
- added L1: 2.2u, Inductor_SMD:L_0805_2012Metric, B.Cu at (37.0, 51.3)
- added L2: 2.2u, Electronics.pretty:IND-SMD_L3.0-W3.0, B.Cu at (37.1, 56.4)
- added R3: 40.2k, Resistor_SMD:R_0201_0603Metric, B.Cu at (30.5, 46.7)
- added R8: 294k, Resistor_SMD:R_0805_2012Metric, B.Cu at (32.6, 57.9)
- added R9: 40.2k, Resistor_SMD:R_0201_0603Metric, B.Cu at (30.5, 51.8)
- added SW1: TS-1187A-B-A-B, Electronics.pretty:SW-SMD_4P-L5.1-W5.1-P3.70-LS6.5-TL-2, F.Cu at (30.6, 64.3)
- added SW2: SK-3296S-01-L3, Electronics.pretty:SW-SMD_SK-3296S-01-L3, F.Cu at (22.2, 59.1)
- added U8: TLV62568DBVR, Electronics.pretty:SOT-23-5_L3.0-W1.7-P0.95-LS2.8-BR, B.Cu at (31.6, 54.0)
- C1, C2: value 10u -> 4.7u; footprint Capacitor_SMD:C_0805_2012Metric -> Capacitor_SMD:C_0402_1005Metric; moved to B.Cu
- C21, C22, C23, C24, C7, U4, U5, U6, U7: moved to B.Cu
- J1: footprint Connector_JST:JST_PH_B2B-PH-SM4-TB_1x02-1MP_P2.00mm_Vertical -> Connector_JST:JST_PH_B2B-PH-K_1x02_P2.00mm_Vertical
- R1: footprint Capacitor_SMD:C_0402_1005Metric -> Resistor_SMD:R_0402_1005Metric
- R2: value DNF -> 180k; footprint Capacitor_SMD:C_0402_1005Metric -> Resistor_SMD:R_0201_0603Metric; moved to B.Cu
- R4, R5, R6, R7: footprint Resistor_SMD:R_2512_6332Metric -> Resistor_SMD:R_0805_2012Metric
- U1: value NCP1117-3.3_SOT223 -> TLV62568DBVR; footprint Package_TO_SOT_SMD:SOT-223-3_TabPin2 -> Electronics.pretty:SOT-23-5_L3.0-W1.7-P0.95-LS2.8-BR; moved to B.Cu
- moved U4 120.4 mm to (27.9, 37.0), turned to 90 degrees
- moved R2 108.9 mm to (34.5, 52.3), turned to 180 degrees
- moved R4 108.3 mm to (32.1, 35.4), turned to -90 degrees
- moved U5 108.3 mm to (37.6, 29.1), turned to 90 degrees
- moved U6 99.4 mm to (46.1, 29.2), turned to -90 degrees
- moved R5 97.9 mm to (41.8, 27.1), turned to -90 degrees
- moved J1 97.8 mm to (21.9, 49.6)
- moved R6 92.1 mm to (46.5, 30.4)
- moved C7 90.6 mm to (41.3, 46.5), turned to 180 degrees
- moved J3 89.9 mm to (21.3, 30.5), turned to -135 degrees
- moved U3 86.6 mm to (41.1, 41.1)
- moved R1 86.3 mm to (38.4, 51.3)
- moved C13 84.9 mm to (46.2, 35.7)
- moved U1 84.6 mm to (31.8, 48.8)
- moved C1 83.6 mm to (29.0, 55.4), turned to -90 degrees
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Connections:
- net Net-(C6-Pad1) renamed +1V1
- C2 pad 1: +3V3 -> +BATT
- J1 pad 1: +BATT -> Net-(J1-Pad1)
- J5 pad 4: /MTR_1_A -> /MTR_3_A
- J5 pad 5: /MTR_1_B -> /MTR_3_B
- J6 pad 4: /MTR_2_A -> /MTR_4_A
- J6 pad 5: /MTR_2_B -> /MTR_4_B
- R1 pad 1: /QSPI_SS -> +3V3
- R1 pad 2: /~{USB_BOOT} -> /RESET
- R2 pad 2: /QSPI_SS -> Net-(R2-Pad2)
- U1 pad 1: GND -> +BATT
- U1 pad 2: +3V3 -> GND
- U1 pad 3: +BATT -> Net-(L1-Pad1)
- U3 pad 11: /MTR_4_A -> /MTR_1_A
- U3 pad 12: /MTR_4_B -> /MTR_1_B
- U3 pad 13: /MTR_1_IN1 -> /MTR_1_IN2
- U3 pad 14: /MTR_1_IN2 -> /MTR_1_IN1
- U3 pad 15: /MTR_2_IN1 -> /MTR_2_IN2
- U3 pad 16: /MTR_2_IN2 -> /MTR_2_IN1
- U3 pad 17: /MTR_3_IN1 -> /MTR_3_IN2
- U3 pad 18: /MTR_3_IN2 -> /MTR_3_IN1
- U3 pad 21: /XOUT -> unconnected-(U3-Pad21)
- U3 pad 26: /RUN -> /RESET
- U3 pad 4: /MTR_1_A -> /MTR_4_A
- U3 pad 5: /MTR_1_B -> /MTR_4_B
- U3 pad 6: /MTR_2_A -> /MTR_3_A
- U3 pad 7: /MTR_2_B -> /MTR_3_B
- U3 pad 8: /MTR_3_A -> /MTR_2_A
- U3 pad 9: /MTR_3_B -> /MTR_2_B
- U6 pad 2: /MTR_1_IN2 -> /MTR_3_IN2
- U6 pad 3: /MTR_1_IN1 -> /MTR_3_IN1
- U7 pad 2: /MTR_2_IN2 -> /MTR_4_IN2
- U7 pad 3: /MTR_2_IN1 -> /MTR_4_IN1
Routing:
- net +5V: track 0.00 -> 150.0 mm, vias 0 -> 5
- net +3V3: track 0.00 -> 148.6 mm, vias 0 -> 8
- net GND: track 0.00 -> 135.9 mm, vias 0 -> 17
- net /QSPI_SCLK: track 0.00 -> 46.4 mm, vias 0 -> 2
- net /QSPI_SD0: track 0.00 -> 40.1 mm, vias 0 -> 2
- net /QSPI_SD2: track 0.00 -> 33.8 mm, vias 0 -> 2
- net /QSPI_SD1: track 0.00 -> 31.3 mm, vias 0 -> 2
- net /MTR_3_IN1: track 0.00 -> 30.9 mm, vias 0 -> 1
- net /MTR_4_B: track 0.00 -> 30.5 mm, vias 0 -> 2
- net +BATT: track 0.00 -> 30.3 mm, vias 0 -> 1
- net /MTR_4_A: track 0.00 -> 29.3 mm, vias 0 -> 2
- net /QSPI_SS: track 0.00 -> 29.0 mm, vias 0 -> 2
- net /MTR_3_B: track 0.00 -> 27.7 mm
- net /MTR_3_IN2: track 0.00 -> 27.0 mm, vias 0 -> 1
- net /MTR_3_A: track 0.00 -> 26.5 mm
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- added copper zone on F.Cu, net +1V1
- added copper zone on F.Cu, net +3V3
- added copper zone on In1.Cu, net GND
Other:
- board outline added: 58 x 58 mm
- copper layers 2 -> 4

Commit message: Adding files
Parts:
- removed C17, C18, C19, C20: 0.22u, Resistor_SMD:R_0201_0603Metric
- added J2: Conn_01x04, Connector_PinHeader_1.27mm:PinHeader_1x04_P1.27mm_Vertical, F.Cu at (39.8, 61.1)
- added J7: Conn_01x05, Connector_PinHeader_1.27mm:PinHeader_1x05_P1.27mm_Vertical, F.Cu at (65.0, 47.0)
- added JP1: SolderJumper_2_Open, Resistor_SMD:R_0402_1005Metric, F.Cu at (17.3, 46.6)
- added JP2: SolderJumper_2_Open, Resistor_SMD:R_0402_1005Metric, F.Cu at (17.3, 48.6)
- added L3: LQP03TN47NH02D, Electronics.pretty:L0201-RD, F.Cu at (54.7, 60.3)
- added RF1: 1909763-1, Electronics.pretty:ANT-SMD_1909763-1, F.Cu at (54.5, 62.5)
- added U10: QMI8658C, Electronics.pretty:LGA-14_L3.0-W2.5-P0.50-BR, F.Cu at (48.8, 52.3)
- added U11: ATGM336H-5N31, Electronics.pretty:GPSM-SMD_ATGM336H-TR, F.Cu at (57.3, 53.2)
- added U9: BME280, Package_LGA:Bosch_LGA-8_2.5x2.5mm_P0.65mm_ClockwisePinNumbering, F.Cu at (48.1, 56.6)
- C10, C11, C12, C13, C14, C15, C5, C6, C8, C9: moved to B.Cu
- L2: footprint Electronics.pretty:IND-SMD_L3.0-W3.0 -> Inductor_SMD:L_0805_2012Metric
- R8: footprint Resistor_SMD:R_0805_2012Metric -> Resistor_SMD:R_0201_0603Metric
- moved C16 95.0 mm to (36.4, 37.2), turned to 90 degrees
- moved C15 94.2 mm to (40.5, 45.2), turned to 90 degrees
- moved C6 88.5 mm to (40.3, 37.3), turned to -90 degrees
- moved C9 86.3 mm to (45.4, 39.5), turned to 180 degrees
- moved C14 85.7 mm to (42.8, 35.1), turned to 90 degrees
- moved C5 84.0 mm to (32.4, 41.5), turned to 180 degrees
- moved C10 76.0 mm to (42.3, 51.4), turned to 90 degrees
- moved C12 40.1 mm to (44.7, 42.0), turned to 180 degrees
- moved C8 38.8 mm to (43.6, 37.5), turned to -90 degrees
- moved C11 34.8 mm to (45.3, 38.5), turned to 180 degrees
- moved C13 4.37 mm to (42.3, 37.6), turned to -90 degrees
- moved C7 1.44 mm to (42.3, 45.4), turned to 0 degrees
- turned L2 to -90 degrees
Connections:
- C3 pad 1: +3V3 -> Net-(JP2-A)
- C4 pad 1: +5V -> Net-(JP1-A)
- L1 pad 2: +3V3 -> Net-(JP2-A)
- L2 pad 2: +5V -> Net-(JP1-A)
- R2 pad 1: +3V3 -> Net-(JP2-A)
- R8 pad 1: +5V -> Net-(JP1-A)
- U3 pad 27: /MTR_4_IN1 -> /MTR_4_IN2
- U3 pad 28: /MTR_4_IN2 -> /MTR_4_IN1
- U3 pad 29: /GPIO18 -> /SDA
- U3 pad 30: /GPIO19 -> /SCL
- U3 pad 31: /GPIO20 -> /GPS_TXD
- U3 pad 32: /GPIO21 -> /GPS_RXD
- U3 pad 35: /GPIO23 -> /HC12_SET
- U3 pad 36: /GPIO24 -> /HC12_RXD
- U3 pad 37: /GPIO25 -> /HC12_TXD
Routing:
- net +3V3: track 148.6 -> 264.5 mm, vias 8 -> 15
- net GND: track 135.9 -> 195.3 mm, vias 17 -> 22
- net Net-(JP1-A): track 0.00 -> 42.7 mm, vias 0 -> 2
- net Net-(JP2-A): track 0.00 -> 32.8 mm, vias 0 -> 2
- net /HC12_SET: track 0.00 -> 27.9 mm, vias 0 -> 1
- net /MTR_4_IN2: track 0.00 -> 27.6 mm, vias 0 -> 1
- net /HC12_RXD: track 0.00 -> 27.3 mm, vias 0 -> 1
- net /SCL: track 0.00 -> 26.8 mm, vias 0 -> 2
- net /HC12_TXD: track 0.00 -> 26.6 mm, vias 0 -> 1
- net /MTR_4_IN1: track 0.00 -> 26.3 mm, vias 0 -> 1
- net /SDA: track 0.00 -> 25.4 mm, vias 0 -> 2
- net /GPS_RXD: track 0.00 -> 22.3 mm, vias 0 -> 2
- net /GPS_TXD: track 0.00 -> 21.5 mm, vias 0 -> 2
- net /SWCLK: track 0.00 -> 18.1 mm
- net /SWD: track 0.00 -> 17.8 mm
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