File: Electronics/CanSat2023.kicad_sch (KiCad schematic)
At the start: 51 parts, among them J1 Conn_01x02, J3 Conn_01x06, J4 Conn_01x06, J5 Conn_01x06, J6 Conn_01x06, SW1 TS-1187A-B-A-B, SW2 SK-3296S-01-L3, U1 TLV62568DBVR, U2 W25Q128JVS, U3 RP2040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

Commit message: Adding files
Parts:
- added J2: Conn_01x04, Connector_PinHeader_1.27mm:PinHeader_1x04_P1.27mm_Vertical, symbol Connector_Generic:Conn_01x04
- added J7: Conn_01x05, Connector_PinHeader_1.27mm:PinHeader_1x05_P1.27mm_Vertical, symbol Connector_Generic:Conn_01x05
- added JP1, JP2: SolderJumper_2_Open, Resistor_SMD:R_0402_1005Metric, symbol Jumper:SolderJumper_2_Open
- added L3: LQP03TN47NH02D, Electronics.pretty:L0201-RD, symbol Components:LQP03TN47NH02D
- added RF1: 1909763-1, Electronics.pretty:ANT-SMD_1909763-1, symbol Components:1909763-1
- added U10: QMI8658C, Electronics.pretty:LGA-14_L3.0-W2.5-P0.50-BR, symbol Components:QMI8658C
- added U11: ATGM336H-5N31, Electronics.pretty:GPSM-SMD_ATGM336H-TR, symbol Components:ATGM336H-5N31
- added U9: BME280, Package_LGA:Bosch_LGA-8_2.5x2.5mm_P0.65mm_ClockwisePinNumbering, symbol Sensor:BME280
- C1, C2: LCSC (none) -> C368809
- C10, C8: LCSC (none) -> C14445
- C11, C12, C13, C14, C15, C16, C5, C6, C7, C9: LCSC (none) -> C1525
- C21, C22, C23, C24: JLCPCB Rotation Offset (none) -> 180; LCSC (none) -> C97805
- C3, C4: LCSC (none) -> C181043
- J3, J4, J5, J6: LCSC (none) -> C160405
- L1: LCSC (none) -> C479898
- L2: footprint Electronics.pretty:IND-SMD_L3.0-W3.0 -> Inductor_SMD:L_0805_2012Metric; LCSC (none) -> C479898
- R1: LCSC (none) -> C106235
- R2: LCSC (none) -> C295779
- R3, R9: LCSC (none) -> C166207
- R4, R5, R6, R7: LCSC (none) -> C158131
- R8: footprint Resistor_SMD:R_0805_2012Metric -> Resistor_SMD:R_0201_0603Metric; LCSC (none) -> C166254
- U1, U8: JLCPCB Rotation Offset (none) -> 180; LCSC (none) -> C163219
- U2: JLCPCB Rotation Offset (none) -> -90; LCSC (none) -> C97521
- U3: LCSC (none) -> C2040
- U4, U5, U6, U7: JLCPCB Rotation Offset (none) -> -90; LCSC (none) -> C82404
Connections:
- net +3V3: now also J2.1 (Pin_1), J7.1 (Pin_1), JP2.2 (B), U10.12 (CS), U10.5 (VDDIO), U10.8 (VDD), U11.8 (VCC), U9.2 (CSB), U9.5 (SDO), U9.6 (VDDIO), U9.8 (VDD); no longer C3.1, L1.2, R2.1
- net +5V: now also JP1.2 (B); no longer C4.1, L2.2, R8.1
- net GND: now also J2.4 (Pin_4), J7.2 (Pin_2), RF1.2, U10.2 (SDX), U10.3 (SCX), U10.6 (GND), U10.7 (GND), U11.1 (GND), U11.10 (GND), U11.12 (GND), U9.1 (GND), U9.7 (GND)
- net MTR_4_IN1: now also U3.28 (GPIO17); no longer U3.27 (GPIO16)
- net MTR_4_IN2: now also U3.27 (GPIO16); no longer U3.28 (GPIO17)
- net SWCLK: now also J2.2 (Pin_2)
- net SWD: now also J2.3 (Pin_3)
- net GPIO18 renamed SDA
- net SDA: now also U10.14 (SDA), U9.3 (SDI)
- net GPIO19 renamed SCL
- net SCL: now also U10.13 (SCL), U9.4 (SCK)
- net GPIO20 renamed GPS_TXD
- net GPS_TXD: now also U11.3 (RXD)
- net GPIO21 renamed GPS_RXD
- net GPS_RXD: now also U11.2 (TXD)
- net GPIO23 renamed HC12_SET
- net HC12_SET: now also J7.5 (Pin_5)
- net GPIO24 renamed HC12_RXD
- net HC12_RXD: now also J7.4 (Pin_4)
- net GPIO25 renamed HC12_TXD
- net HC12_TXD: now also J7.3 (Pin_3)
- new net: C3.1, JP2.1 (A), L1.2, R2.1
- new net: C4.1, JP1.1 (A), L2.2, R8.1
- new net: L3.2, RF1.1, U11.11 (RF_IN)
- new net: L3.1, U11.14 (VCC_RF)
Other:
- note added: "GPS"
- note added: "Gyro and Accel"
- note added: "HC12"
- note added: "SWD"
- note added: "Temp, Pres & Hum"
